File: Eagle/Ganggu.brd (EAGLE design)
At the start: 100 x 50 mm, 50 parts, among them T1 2N2222, T10 2N2222, T11 2N2222, T12 2N2222, T13 2N2222, T14 2N2222, T15 2N2222, T16 2N2222, T2 2N2222, T3 2N2222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

Commit message: More PCB works
Parts:
- added PCB1: PCB_DP_RECTANGLE-50X100, dp_devices:DP10050_V1
- moved U1 99.2 mm to (95.2, 18.4), turned to 90 degrees
- moved T15 5.12 mm to (44.5, 29.7)
- moved T16 5.12 mm to (47.0, 22.1)
- moved R10 5.12 mm to (33.0, 38.6)
- moved R11 5.12 mm to (35.6, 38.6)
- moved R20 5.12 mm to (17.8, 12.5)
- moved R24 5.12 mm to (27.9, 12.5)
- moved R25 5.12 mm to (30.5, 12.5)
- moved R26 5.12 mm to (33.0, 12.5)
- moved R27 5.12 mm to (35.6, 12.5)
- moved R4 5.12 mm to (17.8, 38.6)
- moved R8 5.12 mm to (27.9, 38.6)
- moved R9 5.12 mm to (30.5, 38.6)
- moved T4 5.12 mm to (16.5, 22.1)
- moved T8 5.12 mm to (26.7, 22.1)
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Other:
- outline, holes or cut-outs redrawn
