File: Eagle/Ganggu.sch (EAGLE design)
At the start: 50 parts, among them T1 2N2222, T10 2N2222, T11 2N2222, T12 2N2222, T13 2N2222, T14 2N2222, T15 2N2222, T16 2N2222, T2 2N2222, T3 2N2222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

Commit message: More PCB works
Parts:
- added PCB1: PCB_DP_RECTANGLE-50X100, dp_devices:PCB_DP_RECTANGLE-50X100
Changed lines of the file:
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@@
 <part name="JP1" library="adafruit" deviceset="PINHD-1X18" device=""/>
 <part name="U1" library="SmallRoomLabs_uC" deviceset="PIC16F1829-I/P" device=""/>
+<part name="PCB1" library="dp_devices" deviceset="PCB_DP_RECTANGLE" device="-50X100"/>
 </parts>
 <sheets>
@@
 <instance part="JP1" gate="A" x="78.74" y="99.06" rot="R90"/>
 <instance part="U1" gate="A" x="187.96" y="2.54"/>
+<instance part="PCB1" gate="PCB" x="-25.4" y="78.74"/>
 </instances>
 <busses>
